Commit message: feat: 完成 BUMI3 原生 SONIC 训练与 sim2sim 闭环
具体改动：补齐 BUMI3 质量白名单 30Hz 到 50Hz 严格转换、坐标和 FK 审计、训练样本隔离、TensorBoard 持久化、URDF 碰撞配置、原生 MuJoCo sim2sim、参考影子与验证工具；同时修正 Robot Encoder 参考侧误取 base_link 根姿态的问题，使训练和 sim2sim 均使用 waist_yaw_link FK 锚点。

修改理由与影响：统一 BUMI3 数据、训练和部署的坐标系、频率、关节顺序、MJCF 动力学及腰部锚点契约；保持 SONIC 网络主体、FSQ、PPO、控制频率和 G1/H2 默认行为不变。新增 agent 工作规则，要求代码注释使用详细中文，并在每次修改后完成中文提交、GitHub 推送和 noetix-volc 快进同步。

实际验证：env_isaaclab 下 compileall gear_sonic 通过；四组数据准备、sim2sim 和锚点测试共 24 passed；validate_bumi3_integration.py 通过并确认 21 DoF、22 bodies、sim_dt=0.005、decimation=4、50Hz、action_dim=21、FSQ=64、actor proprioception=690、dynamic decoder 754->21；git diff --cached --check 通过。

未执行项：本轮未提供本地 BUMI3/SMPL 数据路径，因此没有执行 1-env Isaac Lab reset/step；既有服务器完整训练效果也不作为本次静态与单元验证的通过依据。

File: gear_sonic/data/assets/robot_description/urdf/bumi3/bumi.urdf (robot description, URDF)
Before this commit: robot BUMI_V3.0_260119, 22 links, 21 joints
Links:
- link l_knee_pitch_link: geometry collision cylinder length=0.13 radius=0.025; visual mesh filename=../../meshes/bumi3/l_knee_pitch_link.STL
- link l_leg_roll_link: geometry collision cylinder length=0.08 radius=0.03; visual mesh filename=../../meshes/bumi3/l_leg_roll_link.STL
- link r_knee_pitch_link: geometry collision cylinder length=0.13 radius=0.025; visual mesh filename=../../meshes/bumi3/r_knee_pitch_link.STL
- link r_leg_roll_link: geometry collision cylinder length=0.08 radius=0.03; visual mesh filename=../../meshes/bumi3/r_leg_roll_link.STL
